Commit message: version 3 of the workspace - deleted .STL files and replaced with .dae files

File: src/mybot_description/urdf/mybot.xacro (robot description, xacro)
@@ -2,5 +2,5 @@
 <robot name="myrobot" xmlns:xacro="http://www.ros.org/wiki/xacro">
 	  <xacro:property name="cameraSize" value="0.03"/>
-  	  <xacro:property name="cameraMass" value="0.001"/>
+  	  <xacro:property name="cameraMass" value="0.0001"/>
 	  <xacro:include filename="$(find mybot_description)/urdf/mybot.gazebo" />
 	  <xacro:include filename="$(find mybot_description)/urdf/materials.xacro" />
@@ -10,37 +10,34 @@
     <inertial>
       <origin
-        xyz="0.059941 0.20387 0.20658"
-        rpy="0 0 0" />
-      <mass
-        value="1.00" />
-      <inertia
-        ixx="0.018662"
-        ixy="-4.5513E-05"
-        ixz="0.0009887"
-        iyy="0.022098"
-        iyz="0.0003587"
-        izz="0.02544" />
-    </inertial>
-    <visual>
-      <origin
-        xyz="0 0 0"
-        rpy="0 0 0" />
-      <geometry>
-        <mesh
-          filename="package://mybot_description/meshes/chassis.STL" />
-      </geometry>
-      <material
-        name="">
-        <color
-          rgba="0.76863 0.77255 0.76863 1" />
-      </material>
-    </visual>
-    <collision>
-      <origin
-        xyz="0 0 0"
-        rpy="0 0 0" />
-      <geometry>
-        <mesh
-          filename="package://mybot_description/meshes/chassis.STL" />
+        xyz="0.018957 -0.0034534 0.20396"
+        rpy="0 0 0" />
+      <mass
+        value="0.6353" />
+      <inertia
+        ixx="0.018752"
+        ixy="-1.3295E-05"
+        ixz="0.0012594"
+        iyy="0.022099"
+        iyz="0.0003545"
+        izz="0.02535" />
+    </inertial>
+    <visual>
+      <origin
+        xyz="0 0 0"
+        rpy="0 0 0" />
+      <geometry>
+        <mesh
+          filename="package://mybot_description/meshes/chassis.dae" />
+      </geometry>
+      <material name="">
+        <color rgba="0.43922 0.43922 0.43922 1" />
+      </material>
+    </visual>
+    <collision>
+      <origin
+        xyz="0 0 0"
+        rpy="0 0 0" />
+      <geometry>
+        <mesh filename="package://mybot_description/meshes/chassis.dae" />
       </geometry>
     </collision>
@@ -50,37 +47,37 @@
     <inertial>
       <origin
-        xyz="0.0013314 -0.0015346 0.0015292"
-        rpy="0 0 1" />
-      <mass
-        value="0.15984" />
-      <inertia
-        ixx="0.00025061"
-        ixy="8.0674E-09"
-        ixz="6.7668E-07"
-        iyy="0.0002506"
-        iyz="-7.9498E-07"
-        izz="0.00044609" />
-    </inertial>
-    <visual>
-      <origin
-        xyz="0 0 0"
-        rpy="0 0 0" />
-      <geometry>
-        <mesh
-          filename="package://mybot_description/meshes/front_left_wheel.STL" />
-      </geometry>
-      <material
-        name="">
-        <color
-          rgba="0.1098 0.1098 0.1098 1" />
-      </material>
-    </visual>
-    <collision>
-      <origin
-        xyz="0 0 0"
-        rpy="0 0 0" />
-      <geometry>
-        <mesh
-          filename="package://mybot_description/meshes/front_left_wheel.STL" />
+        xyz="-1.6838E-06 3.36E-07 6.9398E-05"
+        rpy="0 0 1" />
+      <mass
+        value="0.15984" />
+      <inertia
+        ixx="0.00025061"
+        ixy="1.0824E-08"
+        ixz="5.5158E-09"
+        iyy="0.0002506"
+        iyz="-2.2109E-08"
+        izz="0.00044609" />
+    </inertial>
+    <visual>
+      <origin
+        xyz="0 0 0"
+        rpy="0 0 0" />
+      <geometry>
+        <mesh
+          filename="package://mybot_description/meshes/front_left_wheel.dae" />
+      </geometry>
+      <material
+        name="">
+        <color
+          rgba="0.1098 0.1098 0.1098 1" />
+      </material>
+    </visual>
+    <collision>
+      <origin
+        xyz="0 0 0"
+        rpy="0 0 0" />
+      <geometry>
+        <mesh
+          filename="package://mybot_description/meshes/front_left_wheel.dae" />
       </geometry>
     </collision>
@@ -90,6 +87,6 @@
     type="continuous">
     <origin
-      xyz="0.27982 0.38747 0.075206"
-      rpy="1.5708 -0.85568 3.1416" />
+      xyz="0.23232 0.18046 0.063906"
+      rpy="1.5708 -0.89583 3.1416" />
     <parent
       link="chassis" />
@@ -100,5 +97,117 @@
     <limit
       effort="1000"
-      velocity="100" />
+      velocity="1500" />
+  </joint>
+  <link
+    name="middle_left_wheel">
+    <inertial>
+      <origin
+        xyz="-1.6618E-06 3.1989E-07 6.9398E-05"
+        rpy="0 0 1" />
+      <mass
+        value="0.15984" />
+      <inertia
+        ixx="0.00025061"
+        ixy="1.0825E-08"
+        ixz="5.5201E-09"
+        iyy="0.0002506"
+        iyz="-2.2123E-08"
+        izz="0.00044609" />
+    </inertial>
+    <visual>
+      <origin
+        xyz="0 0 0"
+        rpy="0 0 0" />
+      <geometry>
+        <mesh
+          filename="package://mybot_description/meshes/middle_left_wheel.dae" />
+      </geometry>
+      <material
+        name="">
+        <color
+          rgba="0.1098 0.1098 0.1098 1" />
+      </material>
+    </visual>
+    <collision>
+      <origin
+        xyz="0 0 0"
+        rpy="0 0 0" />
+      <geometry>
+        <mesh
+          filename="package://mybot_description/meshes/middle_left_wheel.dae" />
+      </geometry>
+    </collision>
+  </link>
+  <joint
+    name="middle_left_wheel_hinge"
+    type="continuous">
+    <origin
+      xyz="0.0024254 0.17526 0.07597"
+      rpy="-1.5708 0.13003 0" />
+    <parent
+      link="chassis" />
+    <child
+      link="middle_left_wheel" />
+    <axis
+      xyz="0 0 1" />
+    <limit
+      effort="1000"
+      velocity="1500" />
+  </joint>
+  <link
+    name="rear_left_wheel">
+    <inertial>
+      <origin
+        xyz="-1.6618E-06 3.1995E-07 6.9398E-05"
+        rpy="0 0 1" />
+      <mass
+        value="0.15984" />
+      <inertia
+        ixx="0.00025061"
+        ixy="1.0825E-08"
+        ixz="5.5202E-09"
+        iyy="0.0002506"
+        iyz="-2.2123E-08"
+        izz="0.00044609" />
+    </inertial>
+    <visual>
+      <origin
+        xyz="0 0 0"
+        rpy="0 0 0" />
+      <geometry>
+        <mesh
+          filename="package://mybot_description/meshes/rear_left_wheel.dae" />
+      </geometry>
+      <material
+        name="">
+        <color
+          rgba="0.1098 0.1098 0.1098 1" />
+      </material>
+    </visual>
+    <collision>
+      <origin
+        xyz="0 0 0"
+        rpy="0 0 0" />
+      <geometry>
+        <mesh
+          filename="package://mybot_description/meshes/rear_left_wheel.dae" />
+      </geometry>
+    </collision>
+  </link>
+  <joint
+    name="rear_left_wheel_hinge"
+    type="continuous">
+    <origin
+      xyz="-0.20669 0.18075 0.10332"
+      rpy="-1.5708 0.13003 0" />
+    <parent
+      link="chassis" />
+    <child
+      link="rear_left_wheel" />
+    <axis
+      xyz="0 0 1" />
+    <limit
+      effort="1000"
+      velocity="1500" />
   </joint>
   <link
@@ -106,37 +215,37 @@
     <inertial>
       <origin
-        xyz="9.3829E-05 0.00013114 -0.0013953"
-        rpy="0 0 1" />
-      <mass
-        value="0.15984" />
-      <inertia
-        ixx="0.00025061"
-        ixy="1.3407E-08"
-        ixz="-5.9803E-07"
-        iyy="0.0002506"
-        iyz="-8.4874E-07"
-        izz="0.00044609" />
-    </inertial>
-    <visual>
-      <origin
-        xyz="0 0 0"
-        rpy="0 0 0" />
-      <geometry>
-        <mesh
-          filename="package://mybot_description/meshes/front_right_wheel.STL" />
-      </geometry>
-      <material
-        name="">
-        <color
-          rgba="0.1098 0.1098 0.1098 1" />
-      </material>
-    </visual>
-    <collision>
-      <origin
-        xyz="0 0 0"
-        rpy="0 0 0" />
-      <geometry>
-        <mesh
-          filename="package://mybot_description/meshes/front_right_wheel.STL" />
+        xyz="-1.6829E-06 3.3642E-07 6.9398E-05"
+        rpy="0 0 1" />
+      <mass
+        value="0.15984" />
+      <inertia
+        ixx="0.00025061"
+        ixy="1.0824E-08"
+        ixz="5.5162E-09"
+        iyy="0.0002506"
+        iyz="-2.2109E-08"
+        izz="0.00044609" />
+    </inertial>
+    <visual>
+      <origin
+        xyz="0 0 0"
+        rpy="0 0 0" />
+      <geometry>
+        <mesh
+          filename="package://mybot_description/meshes/front_right_wheel.dae" />
+      </geometry>
+      <material
+        name="">
+        <color
+          rgba="0.1098 0.1098 0.1098 1" />
+      </material>
+    </visual>
+    <collision>
+      <origin
+        xyz="0 0 0"
+        rpy="0 0 0" />
+      <geometry>
+        <mesh
+          filename="package://mybot_description/meshes/front_right_wheel.dae" />
       </geometry>
     </collision>
@@ -146,6 +255,6 @@
     type="continuous">
     <origin
-      xyz="0.27982 0.030271 0.075206"
-      rpy="-1.5708 -0.94008 3.1416" />
+      xyz="0.23232 -0.17674 0.063906"
+      rpy="-1.5708 -0.98023 3.1416" />
     <parent
       link="chassis" />
@@ -156,61 +265,5 @@
     <limit
       effort="1000"
-      velocity="100" />
-  </joint>
-  <link
-    name="middle_left_wheel">
-    <inertial>
-      <origin
-        xyz="-0.0019962 0.00018008 0.00032398"
-        rpy="0 0 1" />
-      <mass
-        value="0.15984" />
-      <inertia
-        ixx="0.00025062"
-        ixy="1.0458E-08"
-        ixz="-1.0139E-06"
-        iyy="0.0002506"
-        iyz="6.9819E-08"
-        izz="0.00044609" />
-    </inertial>
-    <visual>
-      <origin
-        xyz="0 0 0"
-        rpy="0 0 0" />
-      <geometry>
-        <mesh
-          filename="package://mybot_description/meshes/middle_left_wheel.STL" />
-      </geometry>
-      <material
-        name="">
-        <color
-          rgba="0.1098 0.1098 0.1098 1" />
-      </material>
-    </visual>
-    <collision>
-      <origin
-        xyz="0 0 0"
-        rpy="0 0 0" />
-      <geometry>
-        <mesh
-          filename="package://mybot_description/meshes/middle_left_wheel.STL" />
-      </geometry>
-    </collision>
-  </link>
-  <joint
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